Commit message: Add missing prefix param to parent/child decls for IRB2400 xacro.
Fix #3.

File: abb_common/urdf/irb_2400_macro.xacro (robot description, xacro)
@@ -161,7 +161,7 @@
 			  rpy="0 0 0" />
 			<parent
-			  link="base_link" />
-			<child
-			  link="link_1" />
+			  link="${prefix}base_link" />
+			<child
+			  link="${prefix}link_1" />
 			<axis
 			  xyz="0 0 1" />
@@ -183,7 +183,7 @@
 			  rpy="0 0 0" />
 			<parent
-			  link="link_1" />
-			<child
-			  link="link_2" />
+			  link="${prefix}link_1" />
+			<child
+			  link="${prefix}link_2" />
 			<axis
 			  xyz="0 1 0" />
@@ -205,7 +205,7 @@
 			  rpy="0 0 0" />
 			<parent
-			  link="link_2" />
-			<child
-			  link="link_3" />
+			  link="${prefix}link_2" />
+			<child
+			  link="${prefix}link_3" />
 			<axis
 			  xyz="0 1 0" />
@@ -227,7 +227,7 @@
 			  rpy="0 0 0" />
 			<parent
-			  link="link_3" />
-			<child
-			  link="link_4" />
+			  link="${prefix}link_3" />
+			<child
+			  link="${prefix}link_4" />
 			<axis
 			  xyz="1 0 0" />
@@ -249,7 +249,7 @@
 			  rpy="0 0 0" />
 			<parent
-			  link="link_4" />
-			<child
-			  link="link_5" />
+			  link="${prefix}link_4" />
+			<child
+			  link="${prefix}link_5" />
 			<axis
 			  xyz="0 1 0" />
@@ -271,7 +271,7 @@
 			  rpy="0 0 0" />
 			<parent
-			  link="link_5" />
-			<child
-			  link="link_6" />
+			  link="${prefix}link_5" />
+			<child
+			  link="${prefix}link_6" />
 			<axis
 			  xyz="1 0 0" />
@@ -289,6 +289,6 @@
 		</joint>
 		<joint name="${prefix}joint_6-tool0" type="fixed">
-			<parent link="link_6"/>
-			<child link="tool0"/>
+			<parent link="${prefix}link_6"/>
+			<child link="${prefix}tool0"/>
 			<origin xyz="0 0 0" rpy="0 0 0"/>
 		</joint>
