Commit message: fixed the name of a link for the irb 6600 that was causing a fatal error

File: abb_common/urdf/irb_6600.urdf (robot description, URDF)
Before this commit: robot irb_6600, 7 links, 6 joints
Joints:
- joint joint_1: parent base -> base_link

File: abb_common/urdf/irb_6600_macro.xacro (robot description, xacro)
@@ -89,5 +89,5 @@
   <!--joint list-->
   <joint name="${prefix}joint_1" type="revolute">
-    <parent link="${prefix}base"/>
+    <parent link="${prefix}base_link"/>
     <child link="${prefix}link_1"/>
     <origin xyz="0 0 0" />

Commit message: removed dependency on color image files, and corrected some misnamed files

File: abb_common/urdf/irb_6600.urdf (robot description, URDF)
Before this commit: robot irb_6600, 7 links, 6 joints
Links:
- link base_link: geometry collision mesh filename=package://abb_common/meshes/irb_6600/collision/base_link.dae; visual mesh filename=package://abb_common/meshes/irb_6600/visual/base_link.dae
- link link_1: geometry collision mesh filename=package://abb_common/meshes/irb_6600/collision/link_1.dae; visual mesh filename=package://abb_common/meshes/irb_6600/visual/link_1.dae
- link link_2: geometry collision mesh filename=package://abb_common/meshes/irb_6600/collision/link_2.dae; visual mesh filename=package://abb_common/meshes/irb_6600/visual/link_2.dae
- link link_3: geometry collision mesh filename=package://abb_common/meshes/irb_6600/collision/link_3.dae; visual mesh filename=package://abb_common/meshes/irb_6600/visual/link_3.dae
- link link_4: geometry collision mesh filename=package://abb_common/meshes/irb_6600/collision/link_4.dae; visual mesh filename=package://abb_common/meshes/irb_6600/visual/link_4.dae
- link link_5: geometry collision mesh filename=package://abb_common/meshes/irb_6600/collision/link_5.dae; visual mesh filename=package://abb_common/meshes/irb_6600/visual/link_5.dae
- link link_6: geometry collision mesh filename=package://abb_common/meshes/irb_6600/collision/link_6.dae; visual mesh filename=package://abb_common/meshes/irb_6600/visual/link_6.dae

File: abb_common/urdf/irb_6600_macro.xacro (robot description, xacro)
@@ -2,17 +2,23 @@
 <robot xmlns:xacro="http://ros.org/wiki/xacro">
 <xacro:macro name="irb_6600" params="prefix">
-  <!--link list-->
   <link name="${prefix}base_link">
     <visual>
       <geometry>
-        <mesh filename="package://abb_common/meshes/irb_6600/visual/base.dae" />
+        <mesh filename="package://abb_common/meshes/irb_6600/visual/base_link.dae" />
       </geometry>
     </visual>
     <collision>
       <geometry>
-        <mesh filename="package://abb_common/meshes/irb_6600/collision/base_collision.dae" />
+        <mesh filename="package://abb_common/meshes/irb_6600/collision/base_link.dae" />
       </geometry>
     </collision>
   </link>
+  <joint name="${prefix}joint_1" type="revolute">
+    <parent link="${prefix}base_link"/>
+    <child link="${prefix}link_1"/>
+    <origin xyz="0 0 0" />
+    <axis xyz="0 0 1" />
+    <limit effort="1000" lower="-3.142" upper="3.142" velocity="1.92" />
+  </joint>
   <link name="${prefix}link_1">
     <visual>
@@ -23,8 +29,15 @@
     <collision>
       <geometry>
-        <mesh filename="package://abb_common/meshes/irb_6600/collision/link_1_collision.dae" />
+        <mesh filename="package://abb_common/meshes/irb_6600/collision/link_1.dae" />
       </geometry>
     </collision>
   </link>
+  <joint name="${prefix}joint_2" type="revolute">
+    <parent link="${prefix}link_1"/>
+    <child link="${prefix}link_2"/>
+    <origin xyz="0.32 0 0.78" />
+    <axis xyz="0 1 0" />
+    <limit effort="1000" lower="-1.134" upper="1.396" velocity="1.571" />
+  </joint>
   <link name="${prefix}link_2">
     <visual>
@@ -35,8 +48,15 @@
     <collision>
       <geometry>
-        <mesh filename="package://abb_common/meshes/irb_6600/collision/link_2_collision.dae" />
+        <mesh filename="package://abb_common/meshes/irb_6600/collision/link_2.dae" />
       </geometry>
     </collision>
   </link>
+  <joint name="${prefix}joint_3" type="revolute">
+    <parent link="${prefix}link_2"/>
+    <child link="${prefix}link_3"/>
+    <origin xyz="0 0 1.075" />
+    <axis xyz="0 1 0" />
+    <limit effort="1000" lower="-3.142" upper="1.047" velocity="1.571" />
+  </joint>
   <link name="${prefix}link_3">
     <visual>
@@ -47,8 +67,15 @@
     <collision>
       <geometry>
-        <mesh filename="package://abb_common/meshes/irb_6600/collision/link_3_collision.dae" />
+        <mesh filename="package://abb_common/meshes/irb_6600/collision/link_3.dae" />
       </geometry>
     </collision>
   </link>
+  <joint name="${prefix}joint_4" type="revolute">
+    <parent link="${prefix}link_3"/>
+    <child link="${prefix}link_4"/>
+    <origin xyz="0 0 0.2" />
+    <axis xyz="1 0 0" />
+    <limit effort="1000" lower="-5.24" upper="5.24" velocity="2.618" />
+  </joint>
   <link name="${prefix}link_4">
     <visual>
@@ -59,8 +86,15 @@
     <collision>
       <geometry>
-        <mesh filename="package://abb_common/meshes/irb_6600/collision/link_4_collision.dae" />
+        <mesh filename="package://abb_common/meshes/irb_6600/collision/link_4.dae" />
       </geometry>
     </collision>
   </link>
+  <joint name="${prefix}joint_5" type="revolute">
+    <parent link="${prefix}link_4"/>
+    <child link="${prefix}link_5"/>
+    <origin xyz="1.142 0 0" />
+    <axis xyz="0 1 0" />
+    <limit effort="1000" lower="-2.094" upper="2.094" velocity="2.094"/>
+  </joint>
   <link name="${prefix}link_5">
     <visual>
@@ -71,8 +105,15 @@
     <collision>
       <geometry>
-        <mesh filename="package://abb_common/meshes/irb_6600/collision/link_5_collision.dae" />
+        <mesh filename="package://abb_common/meshes/irb_6600/collision/link_5.dae" />
       </geometry>
     </collision>
   </link>
+  <joint name="${prefix}joint_6" type="revolute">
+    <parent link="${prefix}link_5"/>
+    <child link="${prefix}link_6"/>
+    <origin xyz="0.2 0 0" />
+    <axis xyz="1 0 0" />
+    <limit effort="1000" lower="-5.24" upper="5.24" velocity="3.316"/>
+  </joint>
   <link name="${prefix}link_6">
     <visual>
@@ -83,51 +124,8 @@
     <collision>
       <geometry>
-        <mesh filename="package://abb_common/meshes/irb_6600/collision/link_6_collision.dae" />
+        <mesh filename="package://abb_common/meshes/irb_6600/collision/link_6.dae" />
       </geometry>
     </collision>
   </link>
-  <!--joint list-->
-  <joint name="${prefix}joint_1" type="revolute">
-    <parent link="${prefix}base_link"/>
-    <child link="${prefix}link_1"/>
-    <origin xyz="0 0 0" />
-    <axis xyz="0 0 1" />
-    <limit effort="1000" lower="-3.142" upper="3.142" velocity="1.92" />
-  </joint>
-  <joint name="${prefix}joint_2" type="revolute">
-    <parent link="${prefix}link_1"/>
-    <child link="${prefix}link_2"/>
-    <origin xyz="0.32 0 0.78" />
-    <axis xyz="0 1 0" />
-    <limit effort="1000" lower="-1.134" upper="1.396" velocity="1.571" />
-  </joint>
-  <joint name="${prefix}joint_3" type="revolute">
-    <parent link="${prefix}link_2"/>
-    <child link="${prefix}link_3"/>
-    <origin xyz="0 0 1.075" />
-    <axis xyz="0 1 0" />
-    <limit effort="1000" lower="-3.142" upper="1.047" velocity="1.571" />
-  </joint>
-  <joint name="${prefix}joint_4" type="revolute">
-    <parent link="${prefix}link_3"/>
-    <child link="${prefix}link_4"/>
-    <origin xyz="0 0 0.2" />
-    <axis xyz="1 0 0" />
-    <limit effort="1000" lower="-5.24" upper="5.24" velocity="2.618" />
-  </joint>
-  <joint name="${prefix}joint_5" type="revolute">
-    <parent link="${prefix}link_4"/>
-    <child link="${prefix}link_5"/>
-    <origin xyz="1.142 0 0" />
-    <axis xyz="0 1 0" />
-    <limit effort="1000" lower="-2.094" upper="2.094" velocity="2.094"/>
-  </joint>
-  <joint name="${prefix}joint_6" type="revolute">
-    <parent link="${prefix}link_5"/>
-    <child link="${prefix}link_6"/>
-    <origin xyz="0.2 0 0" />
-    <axis xyz="1 0 0" />
-    <limit effort="1000" lower="-5.24" upper="5.24" velocity="3.316"/>
-  </joint>
 </xacro:macro>
 </robot>
