Commit message: changed naming link_base into base_link and corrected collision meshes

File: abb_common/urdf/irb_6640.urdf (robot description, URDF)
Before this commit: robot irb_6640, 10 links, 9 joints
Links:
- removed link link_base
- added link base_link; collision mesh filename=package://abb_common/meshes/irb_6640/collision/BASE_LINK.stl; visual mesh filename=package://abb_common/meshes/irb_6640/visual/BASE_LINK.stl
Joints:
- joint joint_1: parent link_base -> base_link

File: abb_common/urdf/irb_6640_macro.xacro (robot description, xacro)
@@ -3,8 +3,8 @@
 	<xacro:macro name="irb_6640" params="prefix" >
 		<!-- link list -->
-<link name="${prefix}link_base">
+<link name="${prefix}base_link">
    <collision name="collision">
        <geometry>
-         <mesh filename="package://abb_common/meshes/irb_6640/collision/LINK_BASE.stl"/>
+         <mesh filename="package://abb_common/meshes/irb_6640/collision/BASE_LINK.stl"/>
        </geometry>
         <material name="yellow">
@@ -14,5 +14,5 @@
      <visual name="visual">
        <geometry>
-         <mesh filename="package://abb_common/meshes/irb_6640/visual/LINK_BASE.stl"/>
+         <mesh filename="package://abb_common/meshes/irb_6640/visual/BASE_LINK.stl"/>
        </geometry>
         <material name="orange">
@@ -140,6 +140,5 @@
     <origin xyz="0 0 0.227" rpy="0 0 0"/>
     <axis xyz="0 0 1"/>
-    <parent link="${prefix}link_base"/>
-    <child link="${prefix}link_1"/>
+    <parent link="${prefix}base_link">
     <limit effort="0" lower="-2.967" upper="2.967" velocity="1.7453"/>
   </joint>
