Commit message: common: irb 6640: close empty parent tag. Fix #21.

File: abb_common/urdf/irb_6640_macro.xacro (robot description, xacro)
@@ -140,5 +140,5 @@
     <origin xyz="0 0 0.227" rpy="0 0 0"/>
     <axis xyz="0 0 1"/>
-    <parent link="${prefix}base_link">
+    <parent link="${prefix}base_link"/>
     <limit effort="0" lower="-2.967" upper="2.967" velocity="1.7453"/>
   </joint>

Commit message: common: irb 6640: add missing child link to joint_1.

File: abb_common/urdf/irb_6640_macro.xacro (robot description, xacro)
@@ -141,4 +141,5 @@
     <axis xyz="0 0 1"/>
     <parent link="${prefix}base_link"/>
+    <child link="${prefix}link_1"/>
     <limit effort="0" lower="-2.967" upper="2.967" velocity="1.7453"/>
   </joint>
