Commit message: Add IRB-1600-1.2 urdf model (WIP)
Corrected dimensions, joint speeds and joint limits according to Product
Specification (3HAC023604-005 rev T)

File: abb_common/urdf/irb_1600_1.2.urdf (robot description, URDF)
Before this commit: robot irb_1600_1.2, 8 links, 7 joints
Joints:
- joint joint_2: origin xyz=0.1 0 0.615 rpy=0 0 0 -> xyz=0.15 0 0.4865 rpy=0 0 0
- joint joint_3: origin xyz=0 0 0.705 rpy=0 0 0 -> xyz=0 0 0.475 rpy=0 0 0
- joint joint_4: origin xyz=0.258 0 0.135 rpy=0 0 0 -> xyz=0.300 0 0 rpy=0 0 0
- joint joint_5: origin xyz=0.497 0 0 rpy=0 0 0 -> xyz=0.300 0 0 rpy=0 0 0
- joint joint_6: origin xyz=0.085 0 0 rpy=0 0 0 -> xyz=0.065 0 0 rpy=0 0 0

File: abb_common/urdf/irb_1600_1.2_macro.xacro (robot description, xacro)
@@ -187,5 +187,5 @@
 		<joint name="${prefix}joint_2" type="revolute">
 			<origin
-			  xyz="0.1 0 0.615"
+			  xyz="0.15 0 0.4865"
 			  rpy="0 0 0" />
 			<parent
@@ -196,8 +196,8 @@
 			  xyz="0 1 0" />
 			<limit
-			  lower="-1.7453"
-			  upper="1.9199"
-			  effort="0"
-			  velocity="2.618" />
+			  lower="-1,0995"
+			  upper="1.9198"
+			  effort="0"
+			  velocity="2.7925" />
 			<calibration
 			  rising="0"
@@ -209,5 +209,5 @@
 		<joint name="${prefix}joint_3" type="revolute">
 			<origin
-			  xyz="0 0 0.705"
+			  xyz="0 0 0.475"
 			  rpy="0 0 0" />
 			<parent
@@ -218,8 +218,8 @@
 			  xyz="0 1 0" />
 			<limit
-			  lower="-1.0472"
-			  upper="1.1345"
-			  effort="0"
-			  velocity="2.618" />
+			  lower="−4,1015"
+			  upper="0,9599"
+			  effort="0"
+			  velocity="2.9670" />
 			<calibration
 			  rising="0"
@@ -231,5 +231,5 @@
 		<joint name="${prefix}joint_4" type="revolute">
 			<origin
-			  xyz="0.258 0 0.135"
+			  xyz="0.300 0 0"
 			  rpy="0 0 0" />
 			<parent
@@ -240,8 +240,8 @@
 			  xyz="1 0 0" />
 			<limit
-			  lower="-3.49"
-			  upper="3.49"
-			  effort="0"
-			  velocity="6.2832" />
+			  lower="3,4906"
+			  upper="3.4906"
+			  effort="0"
+			  velocity="5.5850" />
 			<calibration
 			  rising="0"
@@ -253,5 +253,5 @@
 		<joint name="${prefix}joint_5" type="revolute">
 			<origin
-			  xyz="0.497 0 0"
+			  xyz="0.300 0 0"
 			  rpy="0 0 0" />
 			<parent
@@ -262,8 +262,8 @@
 			  xyz="0 1 0" />
 			<limit
-			  lower="-2.0944"
-			  upper="2.0944"
-			  effort="0"
-			  velocity="6.2832" />
+			  lower="-2.0071"
+			  upper="2.0071"
+			  effort="0"
+			  velocity="6.9813" />
 			<calibration
 			  rising="0"
@@ -275,5 +275,5 @@
 		<joint name="${prefix}joint_6" type="revolute">
 			<origin
-			  xyz="0.085 0 0"
+			  xyz="0.065 0 0"
 			  rpy="0 0 0" />
 			<parent
