Commit message: Add irb 1600 visual and collision STL models

File: abb_common/urdf/irb_1600_12.urdf (robot description, URDF)
Before this commit: robot irb_1600_12, 8 links, 7 joints
Links:
- link base_link: geometry collision mesh filename=package://abb_common/meshes/irb_1600_12/collision/base_link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; visual mesh filename=package://abb_common/meshes/irb_1600_12/visual/base_link.STL
- link link_1: geometry collision mesh filename=package://abb_common/meshes/irb_1600_12/collision/link_1.STL; visual mesh filename=package://abb_common/meshes/irb_1600_12/visual/link_1.STL
- link link_2: geometry collision mesh filename=package://abb_common/meshes/irb_1600_12/collision/link_2.STL; visual mesh filename=package://abb_common/meshes/irb_1600_12/visual/link_2.STL
- link link_3: geometry collision mesh filename=package://abb_common/meshes/irb_1600_12/collision/link_3.STL; visual mesh filename=package://abb_common/meshes/irb_1600_12/visual/link_3.STL
- link link_4: geometry collision mesh filename=package://abb_common/meshes/irb_1600_12/collision/link_4.STL; visual mesh filename=package://abb_common/meshes/irb_1600_12/visual/link_4.STL
- link link_5: geometry collision mesh filename=package://abb_common/meshes/irb_1600_12/collision/link_5.STL; visual mesh filename=package://abb_common/meshes/irb_1600_12/visual/link_5.STL
- link link_6: geometry collision mesh filename=package://abb_common/meshes/irb_1600_12/collision/link_6.STL; visual mesh filename=package://abb_common/meshes/irb_1600_12/visual/link_6.STL

File: abb_common/urdf/irb_1600_12_macro.xacro (robot description, xacro)
@@ -4,5 +4,5 @@
 		<!-- link list -->
 		<link name="${prefix}base_link">
-			<!-- <visual>
+			<visual>
      			<origin
         		xyz="0 0 0"
@@ -10,5 +10,5 @@
       			<geometry>
         			<mesh
-          			filename="package://abb_common/meshes/irb_2400/visual/base_link.STL" />
+          			filename="package://abb_common/meshes/irb_1600_12/visual/base_link.STL" />
       			</geometry>
       			<material
@@ -20,5 +20,5 @@
  			<collision>
 				<geometry>
-					<mesh filename="package://abb_common/meshes/irb_2400/collision/base_link.STL" />
+					<mesh filename="package://abb_common/meshes/irb_1600_12/collision/base_link.STL" />
 				</geometry>
 				<material name="yellow">
@@ -26,8 +26,7 @@
 				</material>
 			</collision>
--->
 		</link>
 		<link name="${prefix}link_1">
-<!--			<visual>
+			<visual>
       			<origin
         			xyz="0 0 0"
@@ -35,5 +34,5 @@
       			<geometry>
         			<mesh
-          			filename="package://abb_common/meshes/irb_2400/visual/link_1.STL" />
+          			filename="package://abb_common/meshes/irb_1600_12/visual/link_1.STL" />
       			</geometry>
       			<material name="abb_orange"/>
@@ -44,5 +43,5 @@
         			rpy="0 0 0" />
 				<geometry>
-					<mesh filename="package://abb_common/meshes/irb_2400/collision/link_1.STL" />
+					<mesh filename="package://abb_common/meshes/irb_1600_12/collision/link_1.STL" />
 				</geometry>
 				<material name="yellow"/>
@@ -51,5 +50,5 @@
 		</link>
 		<link name="${prefix}link_2">
-<!--		    <visual>
+		    <visual>
       			<origin
         			xyz="0 0 0"
@@ -57,5 +56,5 @@
       			<geometry>
         			<mesh
-          			filename="package://abb_common/meshes/irb_2400/visual/link_2.STL" />
+          			filename="package://abb_common/meshes/irb_1600_12/visual/link_2.STL" />
       			</geometry>
       			<material name="abb_orange"/>
@@ -66,12 +65,11 @@
         			rpy="0 0 0" />
 				<geometry>
-					<mesh filename="package://abb_common/meshes/irb_2400/collision/link_2_whole.STL" />
-				</geometry>
-				<material name="yellow"/>
-			</collision>
--->
+					<mesh filename="package://abb_common/meshes/irb_1600_12/collision/link_2.STL" />
+				</geometry>
+				<material name="yellow"/>
+			</collision>
 		</link>
 		<link name="${prefix}link_3">
-<!--			<visual>
+			<visual>
 				<origin
 					xyz="0 0 0"
@@ -79,5 +77,5 @@
 			  	<geometry>
 					<mesh
-				  	filename="package://abb_common/meshes/irb_2400/visual/link_3.STL" />
+				  	filename="package://abb_common/meshes/irb_1600_12/visual/link_3.STL" />
 			  	</geometry>
 			  	<material name="abb_orange"/>
@@ -88,12 +86,11 @@
         			rpy="0 0 0" />
 				<geometry>
-					<mesh filename="package://abb_common/meshes/irb_2400/collision/link_3.STL" />
-				</geometry>
-				<material name="yellow"/>
-			</collision>
--->
+					<mesh filename="package://abb_common/meshes/irb_1600_12/collision/link_3.STL" />
+				</geometry>
+				<material name="yellow"/>
+			</collision>
 		</link>
 		<link name="${prefix}link_4">
-<!--			<visual>
+			<visual>
 				  <origin
 					xyz="0 0 0"
@@ -101,5 +98,5 @@
 				  <geometry>
 					<mesh
-					  filename="package://abb_common/meshes/irb_2400/visual/link_4.STL" />
+					  filename="package://abb_common/meshes/irb_1600_12/visual/link_4.STL" />
 				  </geometry>
 				  <material name="abb_orange"/>
@@ -110,12 +107,11 @@
         			rpy="0 0 0" />
 				<geometry>
-					<mesh filename="package://abb_common/meshes/irb_2400/collision/link_4.STL" />
-				</geometry>
-				<material name="yellow"/>
-			</collision>
--->
+					<mesh filename="package://abb_common/meshes/irb_1600_12/collision/link_4.STL" />
+				</geometry>
+				<material name="yellow"/>
+			</collision>
 		</link>
 		<link name="${prefix}link_5">
-<!--			<visual>
+			<visual>
 				<origin
 					xyz="0 0 0"
@@ -123,5 +119,5 @@
 				<geometry>
 					<mesh
-					  filename="package://abb_common/meshes/irb_2400/visual/link_5.STL" />
+					  filename="package://abb_common/meshes/irb_1600_12/visual/link_5.STL" />
 				</geometry>
 				<material name="abb_orange"/>
@@ -132,12 +128,11 @@
         			rpy="0 0 0" />
 				<geometry>
-					<mesh filename="package://abb_common/meshes/irb_2400/collision/link_5.STL" />
-				</geometry>
-				<material name="yellow"/>
-			</collision>
--->
+					<mesh filename="package://abb_common/meshes/irb_1600_12/collision/link_5.STL" />
+				</geometry>
+				<material name="yellow"/>
+			</collision>
 		</link>
 		<link name="${prefix}link_6">
-<!--			<visual>
+			<visual>
 				<origin
 					xyz="0 0 0"
@@ -145,5 +140,5 @@
 				<geometry>
 					<mesh
-					  filename="package://abb_common/meshes/irb_2400/visual/link_6.STL" />
+					  filename="package://abb_common/meshes/irb_1600_12/visual/link_6.STL" />
 				</geometry>
 				<material name="abb_orange"/>
@@ -154,9 +149,8 @@
         			rpy="0 0 0" />
 				<geometry>
-					<mesh filename="package://abb_common/meshes/irb_2400/collision/link_6.STL" />
-				</geometry>
-				<material name="yellow"/>
-			</collision>
--->
+					<mesh filename="package://abb_common/meshes/irb_1600_12/collision/link_6.STL" />
+				</geometry>
+				<material name="yellow"/>
+			</collision>
 		</link>
 		<link name="${prefix}tool0"/>
