Commit message: update IRB_2400 URDF to correct invalid tool0 offset.  Update ikfast plugins and SRDF to match.
git-svn-id: https://swri-ros-pkg.googlecode.com/svn/trunk@1225 076cdf4d-ed99-c8c1-5d01-9bc0d27e81bd

File: abb_common/urdf/irb_2400.urdf (robot description, URDF)
Before this commit: robot irb_2400, 8 links, 7 joints
Joints:
- joint joint_5: origin xyz=0.497 0 -4.4409E-16 rpy=0 0 0 -> xyz=0.497 0 0 rpy=0 0 0
- joint joint_6: origin xyz=0.085 -4.1563E-17 2.2204E-16 rpy=0 0 0 -> xyz=0.085 0 0 rpy=0 0 0
- joint joint_6-tool0: origin xyz=0.085 0 0 rpy=0 0 0 -> xyz=0 0 0 rpy=0 0 0

File: abb_common/urdf/irb_2400_macro.xacro (robot description, xacro)
@@ -177,9 +177,4 @@
 			  damping="0"
 			  friction="0" />
-<!--			<safety_controller
-			  soft_lower_limit="0"
-			  soft_upper_limit="0"
-			  k_position="0"
-			  k_velocity="0" /> -->
 		</joint>
 		<joint name="${prefix}joint_2" type="revolute">
@@ -204,9 +199,4 @@
 			  damping="0"
 			  friction="0" />
-<!--			<safety_controller
-			  soft_lower_limit="0"
-			  soft_upper_limit="0"
-			  k_position="0"
-			  k_velocity="0" /> -->
   		</joint>
 		<joint name="${prefix}joint_3" type="revolute">
@@ -231,9 +221,4 @@
 			  damping="0"
 			  friction="0" />
-<!--			<safety_controller
-			  soft_lower_limit="0"
-			  soft_upper_limit="0"
-			  k_position="0"
-			  k_velocity="0" /> -->
 		</joint>
 		<joint name="${prefix}joint_4" type="revolute">
@@ -258,9 +243,4 @@
 			  damping="0"
 			  friction="0" />
-<!--			<safety_controller
-			  soft_lower_limit="0"
-			  soft_upper_limit="0"
-			  k_position="0"
-			  k_velocity="0" /> -->
 		</joint>
 		<joint name="${prefix}joint_5" type="revolute">
@@ -285,9 +265,4 @@
 			  damping="0"
 			  friction="0" />
-<!--			<safety_controller
-			  soft_lower_limit="0"
-			  soft_upper_limit="0"
-			  k_position="0"
-			  k_velocity="0" /> -->
 		</joint>
 		<joint name="${prefix}joint_6" type="revolute">
@@ -312,14 +287,9 @@
 			  damping="0"
 			  friction="0" />
-<!--			<safety_controller
-			  soft_lower_limit="0"
-			  soft_upper_limit="0"
-			  k_position="0"
-			  k_velocity="0" /> -->
 		</joint>
 		<joint name="${prefix}joint_6-tool0" type="fixed">
 			<parent link="link_6"/>
 			<child link="tool0"/>
-			<origin xyz="0.085 0 0" rpy="0 0 0"/>
+			<origin xyz="0 0 0" rpy="0 0 0"/>
 		</joint>
 		<!-- end of joint list -->

Commit message: Fix for issue #49: add 'base' link (transform to World) This should not affect existing kinematic plugins or MoveIt configurations:
 - the link is not part of the main kinematic chain
 - the transform is implemented as a fixed joint

File: abb_common/urdf/irb_2400.urdf (robot description, URDF)
Before this commit: robot irb_2400, 8 links, 7 joints
Links:
- added link base
Joints:
- added joint base_link-base: type fixed, parent base_link, child base, origin xyz=0 0 0 rpy=0 0 0

File: abb_common/urdf/irb_2400_macro.xacro (robot description, xacro)
@@ -293,5 +293,12 @@
 			<origin xyz="0 0 0" rpy="0 0 0"/>
 		</joint>
-		<!-- end of joint list -->
+                <!-- end of joint list -->
+                <!-- ROS base_link to ABB World Coordinates transform -->
+                <link name="${prefix}base" />
+                <joint name="${prefix}base_link-base" type="fixed">
+                        <origin xyz="0 0 0" rpy="0 0 0"/>
+                        <parent link="${prefix}base_link"/>
+                        <child link="${prefix}base"/>
+                </joint>
 	</xacro:macro>
 </robot>

File: abb_common/urdf/irb_5400.urdf (robot description, URDF)
Before this commit: robot irb_5400, 9 links, 8 joints
Links:
- added link base
Joints:
- added joint base_link-base: type fixed, parent base_link, child base, origin xyz=0 0 0 rpy=0 0 0

File: abb_common/urdf/irb_5400_macro.xacro (robot description, xacro)
@@ -180,4 +180,11 @@
     </joint>
     <!-- end of joint list -->
+    <!-- ROS base_link to ABB World Coordinates transform -->
+    <link name="${prefix}base" />
+    <joint name="${prefix}base_link-base" type="fixed">
+      <origin xyz="0 0 0" rpy="0 0 0"/>
+      <parent link="${prefix}base_link"/>
+      <child link="${prefix}base"/>
+    </joint>
   </xacro:macro>
 </robot>

File: abb_common/urdf/irb_6640.urdf (robot description, URDF)
Before this commit: robot irb_6640, 10 links, 9 joints
Links:
- added link base
Joints:
- added joint base_link-base: type fixed, parent base_link, child base, origin xyz=0 0 0 rpy=0 0 0

File: abb_common/urdf/irb_6640_macro.xacro (robot description, xacro)
@@ -200,4 +200,11 @@
   </joint>
    <!-- end of joint list -->
+  <!-- ROS base_link to ABB World Coordinates transform -->
+  <link name="${prefix}base" />
+  <joint name="${prefix}base_link-base" type="fixed">
+    <origin xyz="0 0 0" rpy="0 0 0"/>
+    <parent link="${prefix}base_link"/>
+    <child link="${prefix}base"/>
+  </joint>
   </xacro:macro>
 </robot>

File: abb_irb2400_support/urdf/irb2400.urdf (robot description, URDF)
Before this commit: robot abb_irb2400, 8 links, 7 joints
Links:
- added link base
Joints:
- added joint base_link-base: type fixed, parent base_link, child base, origin xyz=0 0 0 rpy=0 0 0

File: abb_irb2400_support/urdf/irb2400_macro.xacro (robot description, xacro)
@@ -181,4 +181,11 @@
     </joint>
     <!-- end of joint list -->
+    <!-- ROS base_link to ABB World Coordinates transform -->
+    <link name="${prefix}base" />
+    <joint name="${prefix}base_link-base" type="fixed">
+        <origin xyz="0 0 0" rpy="0 0 0"/>
+        <parent link="${prefix}base_link"/>
+        <child link="${prefix}base"/>
+    </joint>
 </xacro:macro>
 </robot>

File: abb_irb5400_support/urdf/irb5400.urdf (robot description, URDF)
Before this commit: robot abb_irb5400, 9 links, 8 joints
Links:
- added link base
Joints:
- added joint base_link-base: type fixed, parent base_link, child base, origin xyz=0 0 0 rpy=0 0 0

File: abb_irb5400_support/urdf/irb5400_macro.xacro (robot description, xacro)
@@ -180,4 +180,11 @@
     </joint>
     <!-- end of joint list -->
+    <!-- ROS base_link to ABB World Coordinates transform -->
+    <link name="${prefix}base" />
+    <joint name="${prefix}base_link-base" type="fixed">
+        <origin xyz="0 0 0" rpy="0 0 0"/>
+        <parent link="${prefix}base_link"/>
+        <child link="${prefix}base"/>
+    </joint>
 </xacro:macro>
 </robot>

File: abb_irb6600_support/urdf/irb6640.urdf (robot description, URDF)
Before this commit: robot abb_irb6640, 10 links, 9 joints
Links:
- added link base
Joints:
- added joint base_link-base: type fixed, parent base_link, child base, origin xyz=0 0 0 rpy=0 0 0

File: abb_irb6600_support/urdf/irb6640_macro.xacro (robot description, xacro)
@@ -200,4 +200,11 @@
     </joint>
     <!-- end of joint list -->
+    <!-- ROS base_link to ABB World Coordinates transform -->
+    <link name="${prefix}base" />
+    <joint name="${prefix}base_link-base" type="fixed">
+        <origin xyz="0 0 0" rpy="0 0 0"/>
+        <parent link="${prefix}base_link"/>
+        <child link="${prefix}base"/>
+    </joint>
 </xacro:macro>
 </robot>

Commit message: Fix #32: corrects tool0 to match robot controller for abb_common

File: abb_common/urdf/irb_2400.urdf (robot description, URDF)
Before this commit: robot irb_2400, 9 links, 8 joints
Joints:
- joint joint_6-tool0: origin xyz=0 0 0 rpy=0 0 0 -> xyz=0 0 0 rpy=0 1.57079632679 0

File: abb_common/urdf/irb_2400_macro.xacro (robot description, xacro)
@@ -291,5 +291,5 @@
 			<parent link="${prefix}link_6"/>
 			<child link="${prefix}tool0"/>
-			<origin xyz="0 0 0" rpy="0 0 0"/>
+                        <origin xyz="0 0 0" rpy="0 1.57079632679 0"/>
 		</joint>
                 <!-- end of joint list -->

File: abb_common/urdf/irb_5400.urdf (robot description, URDF)
Before this commit: robot irb_5400, 10 links, 9 joints
Joints:
- joint joint_6-tool0: origin xyz=0.0672 0 -0.0470 rpy=0.0 0.6109 0.0 -> xyz=0 0 0 rpy=0.0 1.57079632679 0.0

File: abb_common/urdf/irb_5400_macro.xacro (robot description, xacro)
@@ -177,5 +177,5 @@
       <parent link="${prefix}link_6" />
       <child link="${prefix}tool0" />
-      <origin xyz="0.0672 0 -0.0470" rpy="0.0 0.6109 0.0" />
+      <origin xyz="0 0 0" rpy="0.0 1.57079632679 0.0" />
     </joint>
     <!-- end of joint list -->

File: abb_common/urdf/irb_6640.urdf (robot description, URDF)
Before this commit: robot irb_6640, 11 links, 10 joints
Joints:
- joint joint_6-tool0: origin xyz=.055 0 0  rpy=0 0 0 -> xyz=.055 0 0  rpy=0 1.57079632679 0

File: abb_common/urdf/irb_6640_macro.xacro (robot description, xacro)
@@ -180,5 +180,5 @@
   </joint>
   <joint type="fixed" name="joint_6-tool0">
-    <origin xyz=".055 0 0 " rpy="0 0 0"/>
+    <origin xyz=".055 0 0 " rpy="0 1.57079632679 0"/>
     <axis xyz="1 0 0"/>
     <parent link="${prefix}link_6"/>

Commit message: Revert changes made by pull request #67

File: abb_common/urdf/irb_2400.urdf (robot description, URDF)
Before this commit: robot irb_2400, 9 links, 8 joints
Joints:
- joint joint_6-tool0: origin xyz=0 0 0 rpy=0 1.57079632679 0 -> xyz=0 0 0 rpy=0 0 0

File: abb_common/urdf/irb_2400.xacro (robot description, xacro)
@@ -2,4 +2,4 @@
 <robot name="irb_2400" xmlns:xacro="http://ros.org/wiki/xacro">
 	<xacro:include filename="$(find abb_common)/urdf/irb_2400_macro.xacro"/>
-	<xacro:irb_2400 prefix=""/>
+        <xacro:irb_2400 prefix=""/>
 </robot>

File: abb_common/urdf/irb_2400_macro.xacro (robot description, xacro)
@@ -1,5 +1,5 @@
 <?xml version="1.0" ?>
 <robot xmlns:xacro="http://ros.org/wiki/xacro">
-	<xacro:macro name="irb_2400" params="prefix">
+        <xacro:macro name="irb_2400" params="prefix">
 		<!-- link list -->
 		<link name="${prefix}base_link">
@@ -291,5 +291,5 @@
 			<parent link="${prefix}link_6"/>
 			<child link="${prefix}tool0"/>
-                        <origin xyz="0 0 0" rpy="0 1.57079632679 0"/>
+                        <origin xyz="0 0 0" rpy="0 0 0"/>
 		</joint>
                 <!-- end of joint list -->

File: abb_common/urdf/irb_5400.urdf (robot description, URDF)
Before this commit: robot irb_5400, 10 links, 9 joints
Joints:
- joint joint_6-tool0: origin xyz=0 0 0 rpy=0.0 1.57079632679 0.0 -> xyz=0.0672 0 -0.0470 rpy=0.0 0.6109 0.0

File: abb_common/urdf/irb_5400.xacro (robot description, xacro)
@@ -2,4 +2,4 @@
 <robot name="irb_5400" xmlns:xacro="http://ros.org/wiki/xacro">
 	<xacro:include filename="$(find abb_common)/urdf/irb_5400_macro.xacro" />
-	<xacro:irb_5400 prefix=""/>
+        <xacro:irb_5400 prefix=""/>
 </robot>

File: abb_common/urdf/irb_5400_macro.xacro (robot description, xacro)
@@ -1,5 +1,5 @@
 <?xml version="1.0" ?>
 <robot xmlns:xacro="http://ros.org/wiki/xacro">
-	<xacro:macro name="irb_5400" params="prefix" >
+        <xacro:macro name="irb_5400" params="prefix" >
 		<!-- link list -->
     <link name="${prefix}base_link">
@@ -177,5 +177,5 @@
       <parent link="${prefix}link_6" />
       <child link="${prefix}tool0" />
-      <origin xyz="0 0 0" rpy="0.0 1.57079632679 0.0" />
+      <origin xyz="0.0672 0 -0.0470" rpy="0.0 0.6109 0.0" />
     </joint>
     <!-- end of joint list -->

File: abb_common/urdf/irb_6640.urdf (robot description, URDF)
Before this commit: robot irb_6640, 11 links, 10 joints
Joints:
- joint joint_6-tool0: origin xyz=.055 0 0  rpy=0 1.57079632679 0 -> xyz=.055 0 0 rpy=0 0 0

File: abb_common/urdf/irb_6640.xacro (robot description, xacro)
@@ -2,4 +2,4 @@
 <robot name="irb_6640" xmlns:xacro="http://ros.org/wiki/xacro">
 	<xacro:include filename="$(find abb_common)/urdf/irb_6640_macro.xacro" />
-	<xacro:irb_6640 prefix=""/>
+        <xacro:irb_6640 prefix=""/>
 </robot>

File: abb_common/urdf/irb_6640_macro.xacro (robot description, xacro)
@@ -1,5 +1,5 @@
 <?xml version="1.0" ?>
 <robot xmlns:xacro="http://ros.org/wiki/xacro">
-	<xacro:macro name="irb_6640" params="prefix" >
+        <xacro:macro name="irb_6640" params="prefix" >
 		<!-- link list -->
 <link name="${prefix}base_link">
@@ -180,5 +180,5 @@
   </joint>
   <joint type="fixed" name="joint_6-tool0">
-    <origin xyz=".055 0 0 " rpy="0 1.57079632679 0"/>
+    <origin xyz=".055 0 0" rpy="0 0 0"/>
     <axis xyz="1 0 0"/>
     <parent link="${prefix}link_6"/>
