Commit message: Backported correct 5400 wrist to deprecated abb_common package

File: abb_common/urdf/irb_5400.urdf (robot description, URDF)
Before this commit: robot irb_5400, 8 links, 7 joints
Links:
- added link link_5b; collision mesh filename=package://abb_common/meshes/irb_5400/collision/LINK_5b.STL; visual mesh filename=package://abb_common/meshes/irb_5400/visual/LINK_5b.STL
Joints:
- added joint joint5b: type revolute, parent link_5, child link_5b, origin xyz=.106246 0 0.074394 rpy=0 -1.2217 0, axis 1 0 0, limit lower=-6.0 upper=6.0 effort=100 velocity=6.1086, mimic joint=joint5 multiplier=-1.0 offset=0
- joint joint6: origin xyz=.106246 0 0.074394 rpy=0 -1.2217 0 -> xyz=0.0672 0 -0.0470 rpy=0 0.6109 0; parent link_5 -> link_5b

File: abb_common/urdf/irb_5400_macro.xacro (robot description, xacro)
@@ -93,4 +93,18 @@
       </collision>
     </link>
+    <link name="${prefix}link_5b">
+        <visual>
+            <geometry>
+                <mesh filename="package://abb_common/meshes/irb_5400/visual/LINK_5b.STL"/>
+            </geometry>
+            <material name="lt_black"/>
+        </visual>
+        <collision>
+            <geometry>
+                <mesh filename="package://abb_common/meshes/irb_5400/collision/LINK_5b.STL"/>
+            </geometry>
+            <material name="yellow"/>
+        </collision>
+    </link>
     <link name="${prefix}link_6">
       <visual>
@@ -145,8 +159,16 @@
       <limit lower="-6.0" upper="6.0" effort="100" velocity="6.1086" />
     </joint>
+    <joint name="${prefix}joint5b" type="revolute">
+        <parent link="${prefix}link_5"/>
+        <child link="${prefix}link_5b"/>
+        <origin xyz=".106246 0 0.074394" rpy="0 -1.2217 0"/>
+        <axis xyz="1 0 0"/>
+        <limit lower="-6.0" upper="6.0" effort="100" velocity="6.1086"/>
+        <mimic joint="joint5" multiplier="-1.0" offset="0"/>
+    </joint>
     <joint name="${prefix}joint6" type="revolute">
-      <parent link="${prefix}link_5"/>
+      <parent link="${prefix}link_5b"/>
       <child link="${prefix}link_6"/>
-      <origin xyz=".106246 0 0.074394" rpy="0 -1.2217 0" />
+      <origin xyz="0.0672 0 -0.0470" rpy="0 0.6109 0" />
       <axis xyz="1 0 0" />
       <limit lower="-6.0" upper="6.0" effort="100" velocity="9.3375" />

Commit message: Fix #71: corrects irb5400 joint_6-tool0 transformation in abb_common

File: abb_common/urdf/irb_5400.urdf (robot description, URDF)
Before this commit: robot irb_5400, 10 links, 9 joints
Joints:
- joint joint_6-tool0: origin xyz=0.0672 0 -0.0470 rpy=0.0 0.6109 0.0 -> xyz=0 0 0 rpy=0 0 0

File: abb_common/urdf/irb_5400_macro.xacro (robot description, xacro)
@@ -177,5 +177,5 @@
       <parent link="${prefix}link_6" />
       <child link="${prefix}tool0" />
-      <origin xyz="0.0672 0 -0.0470" rpy="0.0 0.6109 0.0" />
+      <origin xyz="0 0 0" rpy="0 0 0" />
     </joint>
     <!-- end of joint list -->
