Commit message: Fix #32: corrects tool0 to match robot controller     - A link mount_flange is added in the kinematic chain between link_6 and tool0.   - The link orients the frame to match the robot controller allowing tool0 to match     the robot controller tool0 also.

File: abb_irb2400_support/urdf/irb2400.urdf (robot description, URDF)
Before this commit: robot abb_irb2400, 9 links, 8 joints
Links:
- added link mount_flange
Joints:
- removed joint joint_6-tool0
- added joint joint_6-mount_flange: type fixed, parent link_6, child mount_flange, origin xyz=0 0 0 rpy=0 1.57079632679 0
- added joint mount_flange-tool0: type fixed, parent mount_flange, child tool0, origin xyz=0 0 0 rpy=0 0 0

File: abb_irb2400_support/urdf/irb2400_macro.xacro (robot description, xacro)
@@ -118,4 +118,5 @@
         </collision>
     </link>
+    <link name="${prefix}mount_flange"/>
     <link name="${prefix}tool0"/>
     <!-- end of link list -->
@@ -175,6 +176,11 @@
         <dynamics damping="0" friction="0"/>
     </joint>
-    <joint name="${prefix}joint_6-tool0" type="fixed">
+    <joint name="${prefix}joint_6-mount_flange" type="fixed">
         <parent link="${prefix}link_6"/>
+        <child link="${prefix}mount_flange"/>
+        <origin xyz="0 0 0" rpy="0 1.57079632679 0"/>
+    </joint>
+    <joint name="${prefix}mount_flange-tool0" type="fixed">
+        <parent link="${prefix}mount_flange"/>
         <child link="${prefix}tool0"/>
         <origin xyz="0 0 0" rpy="0 0 0"/>

File: abb_irb5400_support/urdf/irb5400.urdf (robot description, URDF)
Before this commit: robot abb_irb5400, 10 links, 9 joints
Links:
- added link mount_flange
Joints:
- removed joint joint_6-tool0
- added joint joint_6-mount_flange: type fixed, parent link_6, child mount_flange, origin xyz=0 0 0 rpy=0 1.57079632679 0
- added joint mount_flange-tool0: type fixed, parent mount_flange, child tool0, origin xyz=0 0 0 rpy=0 0 0

File: abb_irb5400_support/urdf/irb5400_macro.xacro (robot description, xacro)
@@ -121,4 +121,5 @@
         </collision>
     </link>
+    <link name="${prefix}mount_flange"/>
     <link name="${prefix}tool0"/>
     <!-- end of link list -->
@@ -174,8 +175,13 @@
         <limit lower="-6.0" upper="6.0" effort="100" velocity="9.3375"/>
     </joint>
-    <joint name="${prefix}joint_6-tool0" type="fixed">
+    <joint name="${prefix}joint_6-mount_flange" type="fixed">
         <parent link="${prefix}link_6"/>
+        <child link="${prefix}mount_flange"/>
+        <origin xyz="0 0 0" rpy="0 1.57079632679 0"/>
+    </joint>
+    <joint name="${prefix}mount_flange-tool0" type="fixed">
+        <parent link="${prefix}mount_flange"/>
         <child link="${prefix}tool0"/>
-        <origin xyz="0.0672 0 -0.0470" rpy="0.0 0.6109 0.0"/>
+        <origin xyz="0 0 0" rpy="0 0 0"/>
     </joint>
     <!-- end of joint list -->

File: abb_irb6600_support/urdf/irb6640.urdf (robot description, URDF)
Before this commit: robot abb_irb6640, 11 links, 10 joints
Links:
- added link mount_flange
Joints:
- removed joint joint_6-tool0
- added joint joint_6-mount_flange: type fixed, parent link_6, child mount_flange, origin xyz=.055 0 0 rpy=0 1.57079632679 0
- added joint mount_flange-tool0: type fixed, parent mount_flange, child tool0, origin xyz=0 0 0 rpy=0 0 0

File: abb_irb6600_support/urdf/irb6640_macro.xacro (robot description, xacro)
@@ -105,4 +105,5 @@
         </visual>
     </link>
+    <link name="${prefix}mount_flange"/>
     <link name="${prefix}tool0"/>
     <!--Cylinder and piston -->
@@ -179,9 +180,13 @@
         <limit effort="0" lower="-6.283" upper="6.283" velocity="3.3161"/>
     </joint>
-    <joint type="fixed" name="joint_6-tool0">
-        <origin xyz=".055 0 0 " rpy="0 0 0"/>
-        <axis xyz="1 0 0"/>
+    <joint type="fixed" name="${prefix}joint_6-mount_flange">
         <parent link="${prefix}link_6"/>
+        <child link="${prefix}mount_flange"/>
+        <origin xyz=".055 0 0" rpy="0 1.57079632679 0"/>
+    </joint>
+    <joint type="fixed" name="${prefix}mount_flange-tool0">
+        <parent link="${prefix}mount_flange"/>
         <child link="${prefix}tool0"/>
+        <origin xyz="0 0 0" rpy="0 0 0"/>
     </joint>
     <joint type="fixed" name="${prefix}joint_cylinder">

Commit message: Removed mount_flange link and applied changes to tool0

File: abb_irb2400_support/urdf/irb2400.urdf (robot description, URDF)
Before this commit: robot abb_irb2400, 10 links, 9 joints
Links:
- removed link mount_flange
Joints:
- removed joint joint_6-mount_flange
- removed joint mount_flange-tool0
- added joint joint_6-tool0: type fixed, parent link_6, child tool0, origin xyz=0 0 0 rpy=0 1.57079632679 0

File: abb_irb2400_support/urdf/irb2400_macro.xacro (robot description, xacro)
@@ -118,5 +118,4 @@
         </collision>
     </link>
-    <link name="${prefix}mount_flange"/>
     <link name="${prefix}tool0"/>
     <!-- end of link list -->
@@ -128,6 +127,4 @@
         <axis xyz="0 0 1"/>
         <limit lower="-3.1416" upper="3.1416" effort="0" velocity="2.618"/>
-        <calibration rising="0" falling="0"/>
-        <dynamics damping="0" friction="0"/>
     </joint>
     <joint name="${prefix}joint_2" type="revolute">
@@ -137,6 +134,4 @@
         <axis xyz="0 1 0"/>
         <limit lower="-1.7453" upper="1.9199" effort="0" velocity="2.618"/>
-        <calibration rising="0" falling="0"/>
-        <dynamics damping="0" friction="0"/>
     </joint>
     <joint name="${prefix}joint_3" type="revolute">
@@ -146,6 +141,4 @@
         <axis xyz="0 1 0"/>
         <limit lower="-1.0472" upper="1.1345" effort="0" velocity="2.618"/>
-        <calibration rising="0" falling="0"/>
-        <dynamics damping="0" friction="0"/>
     </joint>
     <joint name="${prefix}joint_4" type="revolute">
@@ -155,6 +148,4 @@
         <axis xyz="1 0 0"/>
         <limit lower="-3.49" upper="3.49" effort="0" velocity="6.2832"/>
-        <calibration rising="0" falling="0"/>
-        <dynamics damping="0" friction="0"/>
     </joint>
     <joint name="${prefix}joint_5" type="revolute">
@@ -164,6 +155,4 @@
         <axis xyz="0 1 0"/>
         <limit lower="-2.0944" upper="2.0944" effort="0" velocity="6.2832"/>
-        <calibration rising="0" falling="0"/>
-        <dynamics damping="0" friction="0"/>
     </joint>
     <joint name="${prefix}joint_6" type="revolute">
@@ -173,16 +162,9 @@
         <axis xyz="1 0 0"/>
         <limit lower="-6.9813" upper="6.9813" effort="0" velocity="7.854"/>
-        <calibration rising="0" falling="0"/>
-        <dynamics damping="0" friction="0"/>
     </joint>
-    <joint name="${prefix}joint_6-mount_flange" type="fixed">
+    <joint name="${prefix}joint_6-tool0" type="fixed">
         <parent link="${prefix}link_6"/>
-        <child link="${prefix}mount_flange"/>
+        <child link="${prefix}tool0"/>
         <origin xyz="0 0 0" rpy="0 1.57079632679 0"/>
-    </joint>
-    <joint name="${prefix}mount_flange-tool0" type="fixed">
-        <parent link="${prefix}mount_flange"/>
-        <child link="${prefix}tool0"/>
-        <origin xyz="0 0 0" rpy="0 0 0"/>
     </joint>
     <!-- end of joint list -->

File: abb_irb5400_support/urdf/irb5400.urdf (robot description, URDF)
Before this commit: robot abb_irb5400, 11 links, 10 joints
Links:
- removed link mount_flange
Joints:
- removed joint joint_6-mount_flange
- removed joint mount_flange-tool0
- added joint joint_6-tool0: type fixed, parent link_6, child tool0, origin xyz=0 0 0 rpy=0 1.57079632679 0

File: abb_irb5400_support/urdf/irb5400_macro.xacro (robot description, xacro)
@@ -121,5 +121,4 @@
         </collision>
     </link>
-    <link name="${prefix}mount_flange"/>
     <link name="${prefix}tool0"/>
     <!-- end of link list -->
@@ -175,13 +174,8 @@
         <limit lower="-6.0" upper="6.0" effort="100" velocity="9.3375"/>
     </joint>
-    <joint name="${prefix}joint_6-mount_flange" type="fixed">
+    <joint name="${prefix}joint_6-tool0" type="fixed">
         <parent link="${prefix}link_6"/>
-        <child link="${prefix}mount_flange"/>
+        <child link="${prefix}tool0"/>
         <origin xyz="0 0 0" rpy="0 1.57079632679 0"/>
-    </joint>
-    <joint name="${prefix}mount_flange-tool0" type="fixed">
-        <parent link="${prefix}mount_flange"/>
-        <child link="${prefix}tool0"/>
-        <origin xyz="0 0 0" rpy="0 0 0"/>
     </joint>
     <!-- end of joint list -->

File: abb_irb6600_support/urdf/irb6640.urdf (robot description, URDF)
Before this commit: robot abb_irb6640, 12 links, 11 joints
Links:
- removed link mount_flange
Joints:
- removed joint joint_6-mount_flange
- removed joint mount_flange-tool0
- added joint joint_6-tool0: type fixed, parent link_6, child tool0, origin xyz=.055 0 0 rpy=0 1.57079632679 0

File: abb_irb6600_support/urdf/irb6640_macro.xacro (robot description, xacro)
@@ -105,5 +105,4 @@
         </visual>
     </link>
-    <link name="${prefix}mount_flange"/>
     <link name="${prefix}tool0"/>
     <!--Cylinder and piston -->
@@ -180,13 +179,8 @@
         <limit effort="0" lower="-6.283" upper="6.283" velocity="3.3161"/>
     </joint>
-    <joint type="fixed" name="${prefix}joint_6-mount_flange">
+    <joint type="fixed" name="${prefix}joint_6-tool0">
         <parent link="${prefix}link_6"/>
-        <child link="${prefix}mount_flange"/>
+        <child link="${prefix}tool0"/>
         <origin xyz=".055 0 0" rpy="0 1.57079632679 0"/>
-    </joint>
-    <joint type="fixed" name="${prefix}mount_flange-tool0">
-        <parent link="${prefix}mount_flange"/>
-        <child link="${prefix}tool0"/>
-        <origin xyz="0 0 0" rpy="0 0 0"/>
     </joint>
     <joint type="fixed" name="${prefix}joint_cylinder">
