Commit message: Update to use abb_resources package

File: abb_irb2400_support/urdf/irb2400_macro.xacro (robot description, xacro)
@@ -1,4 +1,5 @@
 <?xml version="1.0"?>
 <robot xmlns:xacro="http://ros.org/wiki/xacro">
+<xacro:include filename="$(find abb_resources)/urdf/common_materials.xacro"/>
 <xacro:macro name="abb_irb2400" params="prefix">
     <!-- link list -->
@@ -9,4 +10,5 @@
                 <mesh filename="package://abb_irb2400_support/meshes/irb2400/visual/base_link.dae"/>
             </geometry>
+            <xacro:material_abb_orange />
         </visual>
         <collision>
@@ -14,7 +16,5 @@
                 <mesh filename="package://abb_irb2400_support/meshes/irb2400/collision/base_link.stl"/>
             </geometry>
-            <material name="yellow">
-                <color rgba="0 1 1 1"/>
-            </material>
+            <xacro:material_abb_yellow />
         </collision>
     </link>
@@ -25,4 +25,5 @@
                 <mesh filename="package://abb_irb2400_support/meshes/irb2400/visual/link_1.dae"/>
             </geometry>
+            <xacro:material_abb_orange />
         </visual>
         <collision>
@@ -31,5 +32,5 @@
                 <mesh filename="package://abb_irb2400_support/meshes/irb2400/collision/link_1.stl"/>
             </geometry>
-            <material name="yellow"/>
+            <xacro:material_abb_yellow />
         </collision>
     </link>
@@ -40,4 +41,5 @@
                 <mesh filename="package://abb_irb2400_support/meshes/irb2400/visual/link_2.dae"/>
             </geometry>
+            <xacro:material_abb_orange />
         </visual>
         <collision>
@@ -46,5 +48,5 @@
                 <mesh filename="package://abb_irb2400_support/meshes/irb2400/collision/link_2_whole.stl"/>
             </geometry>
-            <material name="yellow"/>
+            <xacro:material_abb_yellow />
         </collision>
     </link>
@@ -55,4 +57,5 @@
                 <mesh filename="package://abb_irb2400_support/meshes/irb2400/visual/link_3.dae"/>
             </geometry>
+            <xacro:material_abb_orange />
         </visual>
         <collision>
@@ -61,5 +64,5 @@
                 <mesh filename="package://abb_irb2400_support/meshes/irb2400/collision/link_3.stl"/>
             </geometry>
-            <material name="yellow"/>
+            <xacro:material_abb_yellow />
         </collision>
     </link>
@@ -70,4 +73,5 @@
                 <mesh filename="package://abb_irb2400_support/meshes/irb2400/visual/link_4.dae"/>
             </geometry>
+            <xacro:material_abb_orange />
         </visual>
         <collision>
@@ -76,5 +80,5 @@
                 <mesh filename="package://abb_irb2400_support/meshes/irb2400/collision/link_4.stl"/>
             </geometry>
-            <material name="yellow"/>
+            <xacro:material_abb_yellow />
         </collision>
     </link>
@@ -85,4 +89,5 @@
                 <mesh filename="package://abb_irb2400_support/meshes/irb2400/visual/link_5.dae"/>
             </geometry>
+            <xacro:material_abb_orange />
         </visual>
         <collision>
@@ -91,5 +96,5 @@
                 <mesh filename="package://abb_irb2400_support/meshes/irb2400/collision/link_5.stl"/>
             </geometry>
-            <material name="yellow"/>
+            <xacro:material_abb_yellow />
         </collision>
     </link>
@@ -100,4 +105,5 @@
                 <mesh filename="package://abb_irb2400_support/meshes/irb2400/visual/link_6.dae"/>
             </geometry>
+            <xacro:material_abb_black />
         </visual>
         <collision>
@@ -106,5 +112,5 @@
                 <mesh filename="package://abb_irb2400_support/meshes/irb2400/collision/link_6.stl"/>
             </geometry>
-            <material name="yellow"/>
+            <xacro:material_abb_yellow />
         </collision>
     </link>

File: abb_irb5400_support/urdf/irb5400_macro.xacro (robot description, xacro)
@@ -1,4 +1,5 @@
 <?xml version="1.0"?>
 <robot xmlns:xacro="http://ros.org/wiki/xacro">
+<xacro:include filename="$(find abb_resources)/urdf/common_materials.xacro"/>
 <xacro:macro name="abb_irb5400" params="prefix">
     <!-- link list -->
@@ -8,4 +9,5 @@
                 <mesh filename="package://abb_irb5400_support/meshes/irb5400/visual/base_link.dae"/>
             </geometry>
+            <xacro:material_abb_orange />
         </visual>
         <collision>
@@ -13,7 +15,5 @@
                 <mesh filename="package://abb_irb5400_support/meshes/irb5400/collision/base_link.stl"/>
             </geometry>
-            <material name="yellow">
-                <color rgba="0 1 1 1"/>
-            </material>
+            <xacro:material_abb_yellow />
         </collision>
     </link>
@@ -23,4 +23,5 @@
                 <mesh filename="package://abb_irb5400_support/meshes/irb5400/visual/link_1.dae"/>
             </geometry>
+            <xacro:material_abb_orange />
         </visual>
         <collision>
@@ -28,5 +29,5 @@
                 <mesh filename="package://abb_irb5400_support/meshes/irb5400/collision/link_1.stl"/>
             </geometry>
-            <material name="yellow"/>
+            <xacro:material_abb_yellow />
         </collision>
     </link>
@@ -36,4 +37,5 @@
                 <mesh filename="package://abb_irb5400_support/meshes/irb5400/visual/link_2.dae"/>
             </geometry>
+            <xacro:material_abb_dark_gray />
         </visual>
         <collision>
@@ -41,5 +43,5 @@
                 <mesh filename="package://abb_irb5400_support/meshes/irb5400/collision/link_2.stl"/>
             </geometry>
-            <material name="yellow"/>
+            <xacro:material_abb_yellow />
         </collision>
     </link>
@@ -49,4 +51,5 @@
                 <mesh filename="package://abb_irb5400_support/meshes/irb5400/visual/link_3.dae"/>
             </geometry>
+            <xacro:material_abb_orange />
         </visual>
         <collision>
@@ -54,5 +57,5 @@
                 <mesh filename="package://abb_irb5400_support/meshes/irb5400/collision/link_3.stl"/>
             </geometry>
-            <material name="yellow"/>
+            <xacro:material_abb_yellow />
         </collision>
     </link>
@@ -62,4 +65,5 @@
                 <mesh filename="package://abb_irb5400_support/meshes/irb5400/visual/link_4.dae"/>
             </geometry>
+            <xacro:material_abb_dark_gray />
         </visual>
         <collision>
@@ -67,5 +71,5 @@
                 <mesh filename="package://abb_irb5400_support/meshes/irb5400/collision/link_4.stl"/>
             </geometry>
-            <material name="yellow"/>
+            <xacro:material_abb_yellow />
         </collision>
     </link>
@@ -75,4 +79,5 @@
                 <mesh filename="package://abb_irb5400_support/meshes/irb5400/visual/link_5.dae"/>
             </geometry>
+            <xacro:material_abb_dark_gray />
         </visual>
         <collision>
@@ -80,5 +85,5 @@
                 <mesh filename="package://abb_irb5400_support/meshes/irb5400/collision/link_5.stl"/>
             </geometry>
-            <material name="yellow"/>
+            <xacro:material_abb_yellow />
         </collision>
     </link>
@@ -88,4 +93,5 @@
                 <mesh filename="package://abb_irb5400_support/meshes/irb5400/visual/link_5b.dae"/>
             </geometry>
+            <xacro:material_abb_dark_gray />
         </visual>
         <collision>
@@ -93,5 +99,5 @@
                 <mesh filename="package://abb_irb5400_support/meshes/irb5400/collision/link_5b.stl"/>
             </geometry>
-            <material name="yellow"/>
+            <xacro:material_abb_yellow />
         </collision>
     </link>
@@ -101,4 +107,5 @@
                 <mesh filename="package://abb_irb5400_support/meshes/irb5400/visual/link_6.dae"/>
             </geometry>
+            <xacro:material_abb_black />
         </visual>
         <collision>
@@ -106,5 +113,5 @@
                 <mesh filename="package://abb_irb5400_support/meshes/irb5400/collision/link_6.stl"/>
             </geometry>
-            <material name="yellow"/>
+            <xacro:material_abb_yellow />
         </collision>
     </link>
