Commit message: Corrected 5400 wrist by adding axis 5 mimic joint

File: abb_irb5400_support/urdf/irb5400.urdf (robot description, URDF)
Before this commit: robot abb_irb5400, 8 links, 7 joints
Links:
- added link link_5b; collision mesh filename=package://abb_irb5400_support/meshes/irb5400/collision/link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; visual mesh filename=package://abb_irb5400_support/meshes/irb5400/visual/link_5b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
Joints:
- added joint joint5b: type revolute, parent link_5, child link_5b, origin xyz=.106246 0 0.074394 rpy=0 -1.2217 0, axis 1 0 0, limit lower=-6.0 upper=6.0 effort=100 velocity=6.1086, mimic joint=joint5 multiplier=-1.0 offset=0
- joint joint6: origin xyz=.106246 0 0.074394 rpy=0 -1.2217 0 -> xyz=0.0672 0 -0.0470 rpy=0 0.6109 0; parent link_5 -> link_5b

File: abb_irb5400_support/urdf/irb5400_macro.xacro (robot description, xacro)
@@ -93,4 +93,18 @@
         </collision>
     </link>
+    <link name="${prefix}link_5b">
+        <visual>
+            <geometry>
+                <mesh filename="package://abb_irb5400_support/meshes/irb5400/visual/link_5b.stl"/>
+            </geometry>
+            <material name="lt_black"/>
+        </visual>
+        <collision>
+            <geometry>
+                <mesh filename="package://abb_irb5400_support/meshes/irb5400/collision/link_5b.stl"/>
+            </geometry>
+            <material name="yellow"/>
+        </collision>
+    </link>
     <link name="${prefix}link_6">
         <visual>
@@ -145,8 +159,16 @@
         <limit lower="-6.0" upper="6.0" effort="100" velocity="6.1086"/>
     </joint>
+    <joint name="${prefix}joint5b" type="revolute">
+        <parent link="${prefix}link_5"/>
+        <child link="${prefix}link_5b"/>
+        <origin xyz=".106246 0 0.074394" rpy="0 -1.2217 0"/>
+        <axis xyz="1 0 0"/>
+        <limit lower="-6.0" upper="6.0" effort="100" velocity="6.1086"/>
+        <mimic joint="joint5" multiplier="-1.0" offset="0"/>
+    </joint>
     <joint name="${prefix}joint6" type="revolute">
-        <parent link="${prefix}link_5"/>
+        <parent link="${prefix}link_5b"/>
         <child link="${prefix}link_6"/>
-        <origin xyz=".106246 0 0.074394" rpy="0 -1.2217 0"/>
+        <origin xyz="0.0672 0 -0.0470" rpy="0 0.6109 0"/>
         <axis xyz="1 0 0"/>
         <limit lower="-6.0" upper="6.0" effort="100" velocity="9.3375"/>

Commit message: updates to the macro

File: abb_irb5400_support/urdf/irb5400.urdf (robot description, URDF)
Before this commit: robot abb_irb5400, 10 links, 9 joints
Joints:
- removed joint joint1
- removed joint joint2
- removed joint joint3
- removed joint joint4
- removed joint joint5
- removed joint joint5b
- removed joint joint6
- added joint joint_1: type revolute, parent base_link, child link_1, origin xyz=0 0 0 rpy=0 0 0, axis 0 0 1, limit lower=-2.617 upper=2.617 effort=100 velocity=2.3911
- added joint joint_2: type revolute, parent link_1, child link_2, origin xyz=0.300 0 0.660 rpy=0 0 0, axis 0 1 0, limit lower=-1.396 upper=1.396 effort=100 velocity=2.3911
- added joint joint_3: type revolute, parent link_2, child link_3, origin xyz=0 0 1.200 rpy=0 0 0, axis 0 1 0, limit lower=-1.308 upper=1.308 effort=100 velocity=2.3911
- added joint joint_4: type revolute, parent link_3, child link_4, origin xyz=1.339 0 0.186 rpy=0 0 0, axis 1 0 0, limit lower=-6.0 upper=6.0 effort=100 velocity=8.1157
- added joint joint_5: type revolute, parent link_4, child link_5, origin xyz=0.0693 0 0 rpy=0 0.6109 0, axis 1 0 0, limit lower=-6.0 upper=6.0 effort=100 velocity=6.1086
- added joint joint_5b: type revolute, parent link_5, child link_5b, origin xyz=.106246 0 0.074394 rpy=0 -1.2217 0, axis 1 0 0, limit lower=-6.0 upper=6.0 effort=100 velocity=6.1086, mimic joint=joint_5 multiplier=-1.0 offset=0
- added joint joint_6: type revolute, parent link_5b, child link_6, origin xyz=0.0672 0 -0.0470 rpy=0 0.6109 0, axis 1 0 0, limit lower=-6.0 upper=6.0 effort=100 velocity=9.3375

File: abb_irb5400_support/urdf/irb5400_macro.xacro (robot description, xacro)
@@ -119,5 +119,5 @@
     <!-- end of link list -->
     <!-- joint list -->
-    <joint name="${prefix}joint1" type="revolute">
+    <joint name="${prefix}joint_1" type="revolute">
         <parent link="${prefix}base_link"/>
         <child link="${prefix}link_1"/>
@@ -126,5 +126,5 @@
         <limit lower="-2.617" upper="2.617" effort="100" velocity="2.3911"/>
     </joint>
-    <joint name="${prefix}joint2" type="revolute">
+    <joint name="${prefix}joint_2" type="revolute">
         <parent link="${prefix}link_1"/>
         <child link="${prefix}link_2"/>
@@ -133,5 +133,5 @@
         <limit lower="-1.396" upper="1.396" effort="100" velocity="2.3911"/>
     </joint>
-    <joint name="${prefix}joint3" type="revolute">
+    <joint name="${prefix}joint_3" type="revolute">
         <parent link="${prefix}link_2"/>
         <child link="${prefix}link_3"/>
@@ -140,5 +140,5 @@
         <limit lower="-1.308" upper="1.308" effort="100" velocity="2.3911"/>
     </joint>
-    <joint name="${prefix}joint4" type="revolute">
+    <joint name="${prefix}joint_4" type="revolute">
         <parent link="${prefix}link_3"/>
         <child link="${prefix}link_4"/>
@@ -147,5 +147,5 @@
         <limit lower="-6.0" upper="6.0" effort="100" velocity="8.1157"/>
     </joint>
-    <joint name="${prefix}joint5" type="revolute">
+    <joint name="${prefix}joint_5" type="revolute">
         <parent link="${prefix}link_4"/>
         <child link="${prefix}link_5"/>
@@ -154,5 +154,5 @@
         <limit lower="-6.0" upper="6.0" effort="100" velocity="6.1086"/>
     </joint>
-    <joint name="${prefix}joint5b" type="revolute">
+    <joint name="${prefix}joint_5b" type="revolute">
         <parent link="${prefix}link_5"/>
         <child link="${prefix}link_5b"/>
@@ -160,7 +160,7 @@
         <axis xyz="1 0 0"/>
         <limit lower="-6.0" upper="6.0" effort="100" velocity="6.1086"/>
-        <mimic joint="joint5" multiplier="-1.0" offset="0"/>
+        <mimic joint="joint_5" multiplier="-1.0" offset="0"/>
     </joint>
-    <joint name="${prefix}joint6" type="revolute">
+    <joint name="${prefix}joint_6" type="revolute">
         <parent link="${prefix}link_5b"/>
         <child link="${prefix}link_6"/>
